File: docs/pcb/controller_board/controller_board.kicad_sch (KiCad schematic)
At the start: 1 part

Commit message: add loader
Other:
- title: (none) -> Flight Controller
Changed lines of the file:
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@@
 	(generator_version "8.0")
 	(paper "A4")
+	(title_block
+		(title "Flight Controller")
+		(date "2024-08-31")
+		(rev "Concept")
+	)
 	(symbol
 		(lib_id "MCU_Module:Maple_Mini")
